File: Lights/Lights.kicad_sch (KiCad schematic)
At the start: 9 parts, among them J1 Conn_01x03, U1 LMC6482

Commit message: Light Layout Lab
Assigned footprints + finished layout and routing
Parts:
- C1, C2: footprint (none) -> Capacitor_SMD:C_0805_2012Metric
- D1: footprint (none) -> LED_THT:LED_D5.0mm
- J1: footprint (none) -> Connector_PinHeader_2.54mm:PinHeader_1x03_P2.54mm_Vertical
- R1, R2, R3: footprint (none) -> Resistor_THT:R_Axial_DIN0204_L3.6mm_D1.6mm_P5.08mm_Horizontal
- RV1: footprint (none) -> Potentiometer_THT:Potentiometer_Vishay_T7-YA_Single_Vertical
- U1: footprint (none) -> Package_DIP:DIP-8_W7.62mm
Other:
- moved on the sheet: C1, J1, U1C
